File: hardware/PasswordKeeper.brd (EAGLE design)
At the start: 59.4 x 40.6 mm, 42 parts, among them U1 ATMEGA32U4TQFP-44, U2 3.3V_REG, Y1 16 MHz

Commit message: HW version 1.2
Parts:
- added TP19: TP_ACT_SIG, SparkFun-Connectors:TP_15TH
- added TP20: TP_TAG_SIG, SparkFun-Connectors:TP_15TH
- C3: value 47uF -> 22uF; device SparkFun-Passives:EIA3528-KIT -> SparkFun-Capacitors:0805
- R5: value 90 -> 140
- R6, R7: value 150 -> 85
- S1: device SparkFun-Switches:TACTILE_SWITCH_SMD_RIGHT_ANGLE -> ZnibbLib:TACTILE_SWITCH_SMD_RIGHT_ANGLE
- TP1, TP10, TP11, TP12, TP13, TP14, TP15, TP16, TP17, TP18, TP2, TP3, TP4, TP5, TP6, TP7, TP8, TP9: device SparkFun-Connectors:PAD.03X.03 -> SparkFun-Connectors:TP_15TH
- moved C3 2.54 mm to (20.3, 33.0), turned to 0 degrees
- moved S1 0.25 mm to (53.3, 1.78)
Connections:
- net 3.3V: now also C3.1; no longer C3.A
- net ACT: now also TP19.P$1
- net BUTTON_1: now also S1.P$2; no longer S1.2
- net GND: now also C3.2, S1.P$1, S1.P$5; no longer C3.C, S1.1
- net TAG: now also TP20.P$1
Routing:
- net 3.3V: track 22.3 -> 25.8 mm
- net ACT: track 42.3 -> 43.9 mm
- net TAG: track 10.2 -> 11.4 mm
- net BUTTON_1: track 49.3 -> 48.6 mm
Other:
- board text added: "TP19"
- board text added: "TP20"
- board text removed: "L_ACT"
- board text removed: "L_PWR"
- board text removed: "L_TAG"
