File: hardware/PasswordKeeper.sch (EAGLE design)
At the start: 42 parts, among them U1 ATMEGA32U4TQFP-44, U2 3.3V_REG, Y1 16 MHz

Commit message: HW version 1.2
Parts:
- added TP19: TP_ACT_SIG, SparkFun-Connectors:TEST-POINTTP_15TH_THRU
- added TP20: TP_TAG_SIG, SparkFun-Connectors:TEST-POINTTP_15TH_THRU
- C3: value 47uF -> 22uF; device SparkFun-Passives:CAP_POL3528-KIT -> SparkFun-Capacitors:22UF-0805-6.3V-20%
- R5: value 90 -> 140
- R6, R7: value 150 -> 85
- S1: device SparkFun-Switches:MOMENTARY-SWITCH-SPST-SMD-RIGHT-ANGLE -> ZnibbLib:TACTILE_SWITCH_MOMENTARY_RIGHT_ANGLE
- TP1, TP10, TP11, TP12, TP13, TP14, TP15, TP16, TP17, TP18, TP2, TP3, TP4, TP5, TP6, TP7, TP8, TP9: device SparkFun-Connectors:TEST-POINT3 -> SparkFun-Connectors:TEST-POINTTP_15TH_THRU
Connections:
- net 3.3V: now also C3.1; no longer C3.+
- net ACT: now also TP19.1
- net BUTTON_1: now also S1.P$2; no longer S1.2
- net GND: now also C3.2, S1.P$1, S1.P$5; no longer C3.-, S1.1
- net TAG: now also TP20.1
Other:
- moved on the sheet: R4, TP18, U$1
